File: Schematic/Pocket/ESP32_VGA_Pocket.brd (EAGLE design)
At the start: 190 x 80 mm, 57 parts, among them IC1 74AC00N, IC3 MCP23017SP

Commit message: Schematic update
Parts:
- added RESET_PIN: PTR1PAD1-17Y, testpad:P1-17Y
Connections:
- net RESET: now also RESET_PIN.TP
Routing:
- net RESET: track 239.0 -> 248.3 mm
Changed lines of the file:
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@@
 <element name="LED_RAM" library="led" package="LED5MM" value="" x="146" y="46" rot="R270"/>
 <element name="LED_KEY" library="led" package="LED5MM" value="" x="154" y="46" rot="R270"/>
+<element name="RESET_PIN" library="testpad" package="P1-17Y" value="PTR1PAD1-17Y" x="15.8" y="53.2" rot="R180">
+<attribute name="TP_SIGNAL_NAME" value="" x="15.8" y="53.2" size="1.778" layer="27" rot="R180" display="off"/>
+</element>
 </elements>
 <signals>
@@
 <wire x1="172" y1="61.4" x2="172.085" y2="61.595" width="0.254" layer="16"/>
 <wire x1="23.8" y1="74.4" x2="23.65" y2="74.27" width="0.254" layer="16"/>
-<wire x1="17.4" y1="67.8" x2="4" y2="54.4" width="0.254" layer="1"/>
+<wire x1="17.4" y1="67.8" x2="9.4" y2="59.8" width="0.254" layer="1"/>
+<wire x1="9.4" y1="59.8" x2="4" y2="54.4" width="0.254" layer="1"/>
 <wire x1="17.4" y1="72.2" x2="17.4" y2="67.8" width="0.254" layer="1"/>
 <wire x1="18.2" y1="73" x2="17.4" y2="72.2" width="0.254" layer="1"/>
@@
 <wire x1="22.4" y1="73" x2="22.4" y2="71.2" width="0.254" layer="1"/>
 <wire x1="28.4" y1="28.6" x2="28.565" y2="28.585" width="0.254" layer="1"/>
+<contactref element="RESET_PIN" pad="TP"/>
+<wire x1="9.4" y1="59.6" x2="15.8" y2="53.2" width="0.254" layer="1"/>
+<wire x1="9.4" y1="59.8" x2="9.4" y2="59.6" width="0.254" layer="1"/>
 </signal>
 <signal name="N$9">
