File: Schematic/Pocket/ESP32_VGA_Pocket.sch (EAGLE design)
At the start: 57 parts, among them IC1 74AC00N, IC3 MCP23017SP

Commit message: Schematic update
Parts:
- added RESET_PIN: PTR1PAD1-17Y, testpad:PTR1PAD1-17Y
Connections:
- net RESET: now also RESET_PIN.TP
Changed lines of the file:
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@@
 <setting verticaltext="up"/>
 </settings>
-<grid distance="1.27" unitdist="mm" unit="mm" style="lines" multiple="1" display="no" altdistance="0.01" altunitdist="inch" altunit="inch"/>
+<grid distance="0.1" unitdist="inch" unit="inch" style="lines" multiple="1" display="no" altdistance="0.01" altunitdist="inch" altunit="inch"/>
 <layers>
 <layer number="1" name="Top" color="4" fill="1" visible="no" active="no"/>
@@
 <part name="P+1" library="supply1" deviceset="VCC" device=""/>
 <part name="VDD28" library="supply1" deviceset="VDD" device=""/>
+<part name="RESET_PIN" library="testpad" deviceset="PTR1" device="PAD1-17Y"/>
 </parts>
 <sheets>
@@
 <instance part="P+1" gate="VCC" x="-7.62" y="-76.2"/>
 <instance part="VDD28" gate="G$1" x="-7.62" y="-87.63" rot="R180"/>
+<instance part="RESET_PIN" gate="G$1" x="-119.38" y="81.28" rot="R90"/>
 </instances>
 <busses>
@@
 <wire x1="-127" y1="66.04" x2="-120.65" y2="66.04" width="0.1524" layer="91"/>
 <pinref part="SV1" gate="G$1" pin="6"/>
-<wire x1="-127" y1="66.04" x2="-127" y2="107.95" width="0.1524" layer="91"/>
+<wire x1="-127" y1="66.04" x2="-127" y2="81.28" width="0.1524" layer="91"/>
+<wire x1="-127" y1="81.28" x2="-127" y2="107.95" width="0.1524" layer="91"/>
 <wire x1="-127" y1="107.95" x2="-199.39" y2="107.95" width="0.1524" layer="91"/>
 <wire x1="-199.39" y1="107.95" x2="-199.39" y2="74.93" width="0.1524" layer="91"/>
@@
 <wire x1="-6.35" y1="107.95" x2="-127" y2="107.95" width="0.1524" layer="91"/>
 <junction x="-127" y="107.95"/>
-</segment>
-</net>
+<pinref part="RESET_PIN" gate="G$1" pin="TP"/>
+<wire x1="-121.92" y1="81.28" x2="-127" y2="81.28" width="0.1524" layer="91"/>
+<junction x="-127" y="81.28"/>
+</segment>
+</net>
